File: simpleBuck/simpleBuck.kicad_pcb (KiCad board)
At the start: 2 copper layers, 27 x 25.8 mm, 19 parts, among them J1 Conn_01x02_Pin, J2 Conn_01x02_Pin, Q1 PMV100EPA, U1 LMR33630ADDA

Commit message: Added silly logo, regenerated gerbers
Parts:
- added G***: LOGO, LOGO, B.Cu at (80.2, 74.2)
